File: KiCadFiles_DriverBoard/HeaterController_ConnectorPanel.kicad_pcb (KiCad board)
At the start: 2 copper layers, 122.4 x 44.8 mm, 21 parts, among them J1 721A, J2 KPJX-PM-4S, J3 JST-PH, Q1 BC847, Q2 DMP6023LE, U1 DC-DC-OPTION

Commit message: Add files via upload
Parts:
- added REF**: Symbol_Barrel_Polarity, Symbol:Symbol_Barrel_Polarity, B.Cu at (88.0, 90.0)
- moved R2 2.29 mm to (165.6, 84.4)
- moved R3 2.18 mm to (162.4, 84.4)
- moved D2 0.95 mm to (170.3, 98.4)
- moved C2 0.74 mm to (101.7, 107.0)
Routing:
- net /PWM: track 31.4 -> 36.1 mm
- net Net-(Q1-B): track 3.15 -> 5.19 mm
- net Net-(D1-K): track 27.1 -> 28.9 mm
- net 0V: track 194.4 -> 196.0 mm
- net +24V: track 190.5 -> 192.0 mm
Other:
- board text added: "+"
- board text added: "-"
- board text added: "- HEATER +"
- board text added: "- SENSOR +"
- board text added: "1"
- board text added: "2"
- board text added: "24V DC IN"
- board text added: "3"
- board text added: "4"
- board text added: "MiniThermaDriver"
- board text removed: "24V DC INPUT"
- board text removed: "HEATER / THERMISTOR"
